Commit message: add: conversao da versao 01

File: src/p3at_simulation/urdf/p3at (cópia).xacro (robot description, xacro)
@@ -11,7 +11,7 @@
   <xacro:property name="axel_offset" value="0.05" /> <!-- Space btw top of beam and the each joint -->
   <!-- Import all Gazebo-customization elements, including Gazebo colors -->
-  <xacro:include filename="$(find p3at_description)/urdf/p3at.gazebo" />
+  <xacro:include filename="$(find p3at_simulation)/urdf/p3at.gazebo" />
   <!-- Import Rviz colors -->
-  <xacro:include filename="$(find p3at_description)/urdf/materials.xacro" />
+  <xacro:include filename="$(find p3at_simulation)/urdf/materials.xacro" />
   <!-- Used for fixing robot to Gazebo 'base_link' -->
   <!--link name="world"/-->
@@ -29,5 +29,5 @@
       <origin rpy="0 0 0" xyz="0 0 0.177"/>
       <geometry name="pioneer_geom">
-        <mesh filename="package://amr_robots_description/meshes/p3at_meshes/chassis.stl"/>
+        <mesh filename="package://p3at_simulation/meshes/p3at_meshes/chassis.stl"/>
       </geometry>
       <material name="ChassisRed">
@@ -38,5 +38,5 @@
       <origin rpy="0 0 0" xyz="0 0 0.177"/>
       <geometry>
-        <mesh filename="package://amr_robots_description/meshes/p3at_meshes/chassis.stl"/>
+        <mesh filename="package://p3at_simulation/meshes/p3at_meshes/chassis.stl"/>
       </geometry>
     </collision>
@@ -55,5 +55,5 @@
       <origin rpy="0 0 0" xyz="0 0 0"/>
       <geometry name="pioneer_geom">
-        <mesh filename="package://amr_robots_description/meshes/p3at_meshes/top.stl"/>
+        <mesh filename="package://p3at_simulation/meshes/p3at_meshes/top.stl"/>
       </geometry>
       <material name="TopBlack">
@@ -80,5 +80,5 @@
       <origin rpy="0 0 0" xyz="0 0 0"/>
       <geometry name="pioneer_geom">
-        <mesh filename="package://amr_robots_description/meshes/p3at_meshes/front_sonar.stl"/>
+        <mesh filename="package://p3at_simulation/meshes/p3at_meshes/front_sonar.stl"/>
       </geometry>
       <material name="SonarYellow">
@@ -104,5 +104,5 @@
       <origin rpy="0 0 0" xyz="0 0 0"/>
       <geometry name="pioneer_geom">
-        <mesh filename="package://amr_robots_description/meshes/p3at_meshes/back_sonar.stl"/>
+        <mesh filename="package://p3at_simulation/meshes/p3at_meshes/back_sonar.stl"/>
       </geometry>
       <material name="SonarYellow">
@@ -129,5 +129,5 @@
       <origin rpy="0 0 0" xyz="0 0 0"/>
       <geometry name="pioneer_geom">
-        <mesh filename="package://amr_robots_description/meshes/p3at_meshes/axle.stl"/>
+        <mesh filename="package://p3at_simulation/meshes/p3at_meshes/axle.stl"/>
       </geometry>
       <material name="AxleGrey">
@@ -153,5 +153,5 @@
       <origin rpy="0 0 0" xyz="0 0 0"/>
       <geometry name="pioneer_geom">
-        <mesh filename="package://amr_robots_description/meshes/p3at_meshes/left_hubcap.stl"/>
+        <mesh filename="package://p3at_simulation/meshes/p3at_meshes/left_hubcap.stl"/>
       </geometry>
       <material name="HubcapYellow">
@@ -178,5 +178,5 @@
       <origin rpy="0 0 0" xyz="0 0 0"/>
       <geometry name="pioneer_geom">
-        <mesh filename="package://amr_robots_description/meshes/p3at_meshes/wheel.stl"/>
+        <mesh filename="package://p3at_simulation/meshes/p3at_meshes/wheel.stl"/>
       </geometry>
       <material name="WheelBlack">
@@ -187,5 +187,5 @@
       <origin rpy="-1.57079635 0 0" xyz="0 0 0"/>
       <geometry>
-        <!--mesh filename="package://amr_robots_description/meshes/p3at_meshes/wheel.stl"/-->
+        <!--mesh filename="package://p3at_simulation/meshes/p3at_meshes/wheel.stl"/-->
         <cylinder length="0.075" radius="0.111"/>
       </geometry>
@@ -214,5 +214,5 @@
       <origin rpy="0 0 0" xyz="0 0 0"/>
       <geometry name="pioneer_geom">
-        <mesh filename="package://amr_robots_description/meshes/p3at_meshes/axle.stl"/>
+        <mesh filename="package://p3at_simulation/meshes/p3at_meshes/axle.stl"/>
       </geometry>
       <material name="AxleGrey">
@@ -223,5 +223,5 @@
       <origin rpy="0 0 0" xyz="0 0 0"/>
       <geometry>
-        <mesh filename="package://amr_robots_description/meshes/p3at_meshes/axle.stl"/>
+        <mesh filename="package://p3at_simulation/meshes/p3at_meshes/axle.stl"/>
       </geometry>
     </collision>
@@ -244,5 +244,5 @@
       <origin rpy="0 0 0" xyz="0 0 0"/>
       <geometry name="pioneer_geom">
-        <mesh filename="package://amr_robots_description/meshes/p3at_meshes/left_hubcap.stl"/>
+        <mesh filename="package://p3at_simulation/meshes/p3at_meshes/left_hubcap.stl"/>
       </geometry>
       <material name="HubcapYellow"/>
@@ -251,5 +251,5 @@
       <origin rpy="0 0 0" xyz="0 0 0"/>
       <geometry>
-        <mesh filename="package://amr_robots_description/meshes/p3at_meshes/left_hubcap.stl"/>
+        <mesh filename="package://p3at_simulation/meshes/p3at_meshes/left_hubcap.stl"/>
       </geometry>
     </collision>
@@ -272,5 +272,5 @@
       <origin rpy="0 0 0" xyz="0 0 0"/>
       <geometry name="pioneer_geom">
-        <mesh filename="package://amr_robots_description/meshes/p3at_meshes/wheel.stl"/>
+        <mesh filename="package://p3at_simulation/meshes/p3at_meshes/wheel.stl"/>
       </geometry>
       <material name="WheelBlack"/>
@@ -279,5 +279,5 @@
       <origin rpy="-1.57079635 0 0" xyz="0 0 0"/>
       <geometry>
-        <!--mesh filename="package://amr_robots_description/meshes/p3at_meshes/wheel.stl"/-->
+        <!--mesh filename="package://p3at_simulation/meshes/p3at_meshes/wheel.stl"/-->
         <cylinder length="0.075" radius="0.111"/>
       </geometry>
@@ -306,5 +306,5 @@
       <origin rpy="0 0 0" xyz="0 0 0"/>
       <geometry name="pioneer_geom">
-        <mesh filename="package://amr_robots_description/meshes/p3at_meshes/axle.stl"/>
+        <mesh filename="package://p3at_simulation/meshes/p3at_meshes/axle.stl"/>
       </geometry>
       <material name="AxleGrey">
@@ -330,5 +330,5 @@
       <origin rpy="0 0 0" xyz="0 0 0"/>
       <geometry name="pioneer_geom">
-        <mesh filename="package://amr_robots_description/meshes/p3at_meshes/right_hubcap.stl"/>
+        <mesh filename="package://p3at_simulation/meshes/p3at_meshes/right_hubcap.stl"/>
       </geometry>
       <material name="HubcapYellow">
@@ -355,5 +355,5 @@
       <origin rpy="0 0 0" xyz="0 0 0"/>
       <geometry name="pioneer_geom">
-        <mesh filename="package://amr_robots_description/meshes/p3at_meshes/wheel.stl"/>
+        <mesh filename="package://p3at_simulation/meshes/p3at_meshes/wheel.stl"/>
       </geometry>
       <material name="WheelBlack">
@@ -364,5 +364,5 @@
       <origin rpy="-1.57079635 0 0" xyz="0 0 0"/>
       <geometry>
-        <!--mesh filename="package://amr_robots_description/meshes/p3at_meshes/wheel.stl"/-->
+        <!--mesh filename="package://p3at_simulation/meshes/p3at_meshes/wheel.stl"/-->
         <cylinder length="0.075" radius="0.111"/>
       </geometry>
@@ -391,5 +391,5 @@
       <origin rpy="0 0 0" xyz="0 0 0"/>
       <geometry name="pioneer_geom">
-        <mesh filename="package://amr_robots_description/meshes/p3at_meshes/axle.stl"/>
+        <mesh filename="package://p3at_simulation/meshes/p3at_meshes/axle.stl"/>
       </geometry>
       <material name="AxleGrey">
@@ -400,5 +400,5 @@
       <origin rpy="0 0 0" xyz="0 0 0"/>
       <geometry>
-        <mesh filename="package://amr_robots_description/meshes/p3at_meshes/axle.stl"/>
+        <mesh filename="package://p3at_simulation/meshes/p3at_meshes/axle.stl"/>
       </geometry>
     </collision>
@@ -421,5 +421,5 @@
       <origin rpy="0 0 0" xyz="0 0 0"/>
       <geometry name="pioneer_geom">
-        <mesh filename="package://amr_robots_description/meshes/p3at_meshes/right_hubcap.stl"/>
+        <mesh filename="package://p3at_simulation/meshes/p3at_meshes/right_hubcap.stl"/>
       </geometry>
       <material name="HubcapYellow"/>
@@ -428,5 +428,5 @@
       <origin rpy="0 0 0" xyz="0 0 0"/>
       <geometry>
-        <mesh filename="package://amr_robots_description/meshes/p3at_meshes/right_hubcap.stl"/>
+        <mesh filename="package://p3at_simulation/meshes/p3at_meshes/right_hubcap.stl"/>
       </geometry>
     </collision>
@@ -449,5 +449,5 @@
       <origin rpy="0 0 0" xyz="0 0 0"/>
       <geometry name="pioneer_geom">
-        <mesh filename="package://amr_robots_description/meshes/p3at_meshes/wheel.stl"/>
+        <mesh filename="package://p3at_simulation/meshes/p3at_meshes/wheel.stl"/>
       </geometry>
       <material name="WheelBlack"/>
@@ -456,5 +456,5 @@
       <origin rpy="-1.57079635 0 0" xyz="0 0 0"/>
       <geometry>
-        <!--mesh filename="package://amr_robots_description/meshes/p3at_meshes/wheel.stl"/-->
+        <!--mesh filename="package://p3at_simulation/meshes/p3at_meshes/wheel.stl"/-->
         <cylinder length="0.075" radius="0.111"/>
       </geometry>
@@ -484,5 +484,5 @@
       <origin xyz="0 0 0" rpy="0 0 0"/>
       <geometry>
-        <mesh filename="package://p3at_description/meshes/hokuyo.dae"/>
+        <mesh filename="package://p3at_simulation/meshes/hokuyo.dae"/>
       </geometry>
     </visual>
@@ -503,5 +503,5 @@
       <origin xyz="0 0 0" rpy="0 0 0"/>
       <geometry>
-        <mesh filename="package://p3at_description/meshes/base_laser.dae"/>
+        <mesh filename="package://p3at_simulation/meshes/base_laser.dae"/>
       </geometry>
     </visual>
@@ -577,5 +577,5 @@
       <geometry>
         <!--cylinder length="0.01" radius="0.02"/-->
-	<mesh filename="package://p3at_description/meshes/base_cam.dae"/>
+	<mesh filename="package://p3at_simulation/meshes/base_cam.dae"/>
       </geometry>
       <material name="red"/>
@@ -596,5 +596,5 @@
       <geometry>
         <!--box size="0.02 0.02 0.02"/-->
-	<mesh filename="package://p3at_description/meshes/pan_cam.dae"/>
+	<mesh filename="package://p3at_simulation/meshes/pan_cam.dae"/>
       </geometry>
       <material name="green"/>
@@ -615,5 +615,5 @@
       <geometry>
         <!--box size="0.02 0.02 0.02"/-->
-	<mesh filename="package://p3at_description/meshes/tilt_cam.dae"/>
+	<mesh filename="package://p3at_simulation/meshes/tilt_cam.dae"/>
       </geometry>
       <material name="ChassisRed">
